File: fpga-banks-16-34.sch (KiCad schematic (older format))
At the start: 13 parts, among them U8 PCA9517ADMR2G

Commit message: Add I2C connector
Parts:
- added J4: 61300211121, rdimm-breakout-footprints:PinHeader_1x2_P2.54_Drill0.9mm, symbol rdimm-breakout:61300211121
- added R1, R2: R_0R_0402, rdimm-breakout-footprints:0402-res, symbol rdimm-breakout:R_0R_0402-rdimm-breakout
- added TP1, TP2: TP_SMD1MM, rdimm-breakout-footprints:Testpoint_smd_1mm, symbol rdimm-breakout:TP_SMD1MM-rdimm-breakout
Connections:
- wire segments 41 -> 49
Other:
- note added: "Bypass I2C"
- note added: "I2C header"
- note added: "IF mounted Do not populate I2C logic translator"
- moved on the sheet: R170
Changed lines of the file:
@@
 Text Notes 6125 4800 0    50   ~ 0
 Default 000
-Text Notes 7500 5675 0    50   ~ 0
+Text Notes 4850 6225 0    50   ~ 0
 Open drain pin
 Wire Wire Line
-	7425 5250 7425 5425
-Text GLabel 7425 5425 3    50   Input ~ 0
+	4775 5800 4775 5975
+Text GLabel 4775 5975 3    50   Input ~ 0
 ~EVENT
 $Comp
 L rdimm-breakout:R_4k7_0402-rdimm-breakout R170
 U 1 1 628AFA47
-P 7425 5100
-F 0 "R170" V 7275 5125 60  0000 L CNN
-F 1 "R_4k7_0402" H 7425 4950 60  0001 C CNN
-F 2 "rdimm-breakout-footprints:0402-res" H 7625 5300 60  0001 L CNN
-F 3 "" H 7425 5100 50  0001 C CNN
-F 4 "VISHAY" H 7625 5500 60  0001 L CNN "Manufacturer"
-F 5 "MCS04020C4701FE000" H 7625 5400 60  0001 L CNN "MPN"
-F 6 "4k7" V 7575 5125 50  0000 L CNN "Val"
-	1    7425 5100
-	0    1    1    0
-$EndComp
-Wire Wire Line
-	7425 4950 7425 4800
+P 4775 5650
+F 0 "R170" V 4625 5675 60  0000 L CNN
+F 1 "R_4k7_0402" H 4775 5500 60  0001 C CNN
+F 2 "rdimm-breakout-footprints:0402-res" H 4975 5850 60  0001 L CNN
+F 3 "" H 4775 5650 50  0001 C CNN
+F 4 "VISHAY" H 4975 6050 60  0001 L CNN "Manufacturer"
+F 5 "MCS04020C4701FE000" H 4975 5950 60  0001 L CNN "MPN"
+F 6 "4k7" V 4925 5675 50  0000 L CNN "Val"
+	1    4775 5650
+	0    1    1    0
+$EndComp
+Wire Wire Line
+	4775 5500 4775 5350
 Text Notes 5625 4700 0    98   ~ 20
 Serial adress select
@@
 Text GLabel 5950 6125 0    50   Input ~ 0
 SA2
-Text GLabel 7425 4800 1    50   Input ~ 0
+Text GLabel 4775 5350 1    50   Input ~ 0
 VDDQ
+Wire Wire Line
+	12925 5100 12225 5100
+Wire Wire Line
+	12925 5000 12225 5000
+Text GLabel 12150 5100 0    50   Input ~ 0
+SDA_1V2
+Text GLabel 12150 5000 0    50   Input ~ 0
+SCL_1V2
+$Comp
+L rdimm-breakout:R_0R_0402-rdimm-breakout R1
+U 1 1 61B29083
+P 9375 6150
+F 0 "R1" H 9075 6250 60  0000 L CNN
+F 1 "R_0R_0402" H 9375 6000 60  0001 C CNN
+F 2 "rdimm-breakout-footprints:0402-res" H 9575 6350 60  0001 L CNN
+F 3 "" H 9375 6150 50  0001 C CNN
+F 4 "PANASONIC" H 9575 6550 60  0001 L CNN "Manufacturer"
+F 5 "ERJ2GE0R00X" H 9575 6450 60  0001 L CNN "MPN"
+F 6 "DNP" H 9300 6150 50  0000 L CNN "DNP"
+	1    9375 6150
+	1    0    0    -1
+$EndComp
+$Comp
+L rdimm-breakout:R_0R_0402-rdimm-breakout R2
+U 1 1 61B2908C
+P 9375 6325
+F 0 "R2" H 9075 6425 60  0000 L CNN
+F 1 "R_0R_0402" H 9375 6175 60  0001 C CNN
+F 2 "rdimm-breakout-footprints:0402-res" H 9575 6525 60  0001 L CNN
+F 3 "" H 9375 6325 50  0001 C CNN
+F 4 "PANASONIC" H 9575 6725 60  0001 L CNN "Manufacturer"
+F 5 "ERJ2GE0R00X" H 9575 6625 60  0001 L CNN "MPN"
+F 6 "DNP" H 9300 6325 50  0000 L CNN "DNP"
+	1    9375 6325
+	1    0    0    -1
+$EndComp
+Wire Notes Line
+	8275 5900 10475 5900
+Wire Notes Line
+	10475 5900 10475 6575
+Wire Notes Line
+	10475 6575 8275 6575
+Wire Notes Line
+	8275 6575 8275 5900
+Text Notes 8375 6000 0    50   ~ 0
+Bypass I2C
+Text Notes 8325 6525 0    39   ~ 0
+IF mounted Do not populate I2C logic translator
+Wire Wire Line
+	9225 6325 8900 6325
+Wire Wire Line
+	9225 6150 8900 6150
+Text GLabel 8900 6325 0    50   Input ~ 0
+SDA_1V2
+Text GLabel 8900 6150 0    50   Input ~ 0
+SCL_1V2
+Wire Wire Line
+	9525 6150 9925 6150
+Wire Wire Line
+	9525 6325 9925 6325
+Text GLabel 9925 6325 2    50   Input ~ 0
+SDA_2V5
+Text GLabel 9925 6150 2    50   Input ~ 0
+SCL_2V5
+Text Notes 12050 4650 0    98   ~ 20
+I2C header
+$Comp
+L rdimm-breakout:TP_SMD1MM-rdimm-breakout TP2
+U 1 1 61B53CB4
+P 12225 5200
+F 0 "TP2" V 12225 5150 50  0000 R CNN
+F 1 "TP_SMD1MM" H 12225 5100 50  0001 C CNN
+F 2 "rdimm-breakout-footprints:Testpoint_smd_1mm" H 12425 5400 60  0001 L CNN
+F 3 "" H 12425 5500 60  0001 L CNN
+	1    12225 5200
+	1    0    0    -1
+$EndComp
+Connection ~ 12225 5100
+Wire Wire Line
+	12225 5100 12150 5100
+$Comp
+L rdimm-breakout:TP_SMD1MM-rdimm-breakout TP1
+U 1 1 61B5478E
+P 12225 4900
+F 0 "TP1" V 12225 4850 50  0000 R CNN
+F 1 "TP_SMD1MM" H 12225 4800 50  0001 C CNN
+F 2 "rdimm-breakout-footprints:Testpoint_smd_1mm" H 12425 5100 60  0001 L CNN
+F 3 "" H 12425 5200 60  0001 L CNN
+	1    12225 4900
+	-1   0    0    1
+$EndComp
+Connection ~ 12225 5000
+Wire Wire Line
+	12225 5000 12150 5000
+$Comp
+L rdimm-breakout:61300211121 J4
+U 1 1 61B5CEFA
+P 13025 5100
+F 0 "J4" V 13116 4972 50  0000 R CNN
+F 1 "61300211121" V 13025 4972 50  0000 R CNN
+F 2 "rdimm-breakout-footprints:PinHeader_1x2_P2.54_Drill0.9mm" H 13225 5300 60  0001 L CNN
+F 3 "https://katalog.we-online.de/em/datasheet/6130xx11121.pdf" H 13225 5400 60  0001 L CNN
+F 4 "61300211121" H 13225 5600 60  0001 L CNN "MPN"
+F 5 "Wurth Electronic" H 13225 6200 60  0001 L CNN "Manufacturer"
+	1    13025 5100
+	0    -1   -1   0
+$EndComp
 $EndSCHEMATC

Commit message: Add FTDI and USB power supply
Parts:
- removed J4: 61300211121, rdimm-breakout-footprints:PinHeader_1x2_P2.54_Drill0.9mm, symbol rdimm-breakout:61300211121
- removed R1, R2: R_0R_0402, rdimm-breakout-footprints:0402-res, symbol rdimm-breakout:R_0R_0402-rdimm-breakout
- removed R171, R172, R173, R174: R_4k7_0402, rdimm-breakout-footprints:0402-res, symbol rdimm-breakout:R_4k7_0402-rdimm-breakout
- added J?: 825437-4, rdimm-breakout-footprints:TE_825437-4, symbol rdimm-breakout:825437-4
- added R?: R_0R_0603, rdimm-breakout-footprints:0603-res, symbol rdimm-breakout:R_0R_0603
- added R? (x4): R_10k_0402, rdimm-breakout-footprints:0402-res, symbol rdimm-breakout:R_10k_0402
Connections:
- net labels added: SCL, SDA, VCC2V5, VCC3V3, V_AUX
- net labels removed: SCL_1V2, SDA_1V2
Other:
- note removed: "Bypass I2C"
- note removed: "IF mounted Do not populate I2C logic translator"
- moved on the sheet: R164, R165, R166, R167, R168, R169, R170, TP1, TP12, TP2, U8

Commit message: Update labels on the schematics
Parts:
- removed J?: 825437-4, rdimm-breakout-footprints:TE_825437-4, symbol rdimm-breakout:825437-4
- added C22, C23: C_100n_0402, rdimm-breakout-footprints:0402-cap, symbol rdimm-breakout:C_100n_0402
- added J4: 0022232041, rdimm-breakout-footprints:PinHeader_1x4_P2.54mm_Drill1.02mm, symbol rdimm-breakout:0022232041
- gave numbers to parts that had none: 5
Connections:
- net labels removed: VDDQ, VDDSPD
Changed lines of the file:
@@
 Wire Wire Line
 	7550 5775 7725 5775
-Text GLabel 7150 5475 0    50   Input ~ 0
-VDDQ
 Wire Wire Line
 	7725 5475 7150 5475
 Wire Wire Line
 	8425 5475 9025 5475
-Text GLabel 9025 5475 2    50   Input ~ 0
-VDDSPD
 Text GLabel 9025 5675 2    50   Input ~ 0
 SDA_2V5
@@
 	11400 5300 11575 5300
 $Comp
-L rdimm-breakout:GND-rdimm-breakout #PWR?
+L rdimm-breakout:GND-rdimm-breakout #PWR0134
 U 1 1 623664C2
 P 11400 5300
-F 0 "#PWR?" H 11400 5050 50  0001 C CNN
+F 0 "#PWR0134" H 11400 5050 50  0001 C CNN
 F 1 "GND" H 11405 5127 50  0000 C CNN
 F 2 "" H 11400 5300 50  0001 C CNN
@@
 	-1   0    0    -1
 $EndComp
-$Comp
-L rdimm-breakout:825437-4 J?
-U 1 1 62367F31
-P 11725 5000
-F 0 "J?" V 11824 4922 50  0000 R CNN
-F 1 "825437-4" V 11915 4922 50  0000 R CNN
-F 2 "rdimm-breakout-footprints:TE_825437-4" H 11925 5300 60  0001 L CNN
-F 3 "https://www.te.com/usa-en/product-825437-4.datasheet.pdf" H 11925 5400 60  0001 L CNN
-F 4 "825437-4" H 11925 5500 60  0001 L CNN "MPN"
-F 5 "TE Connectivity" H 11925 5600 60  0001 L CNN "Manufacturer"
-	1    11725 5000
-	0    -1   1    0
-$EndComp
 Text GLabel 5725 5150 1    50   Input ~ 0
 VCC2V5
@@
 V_AUX
 $Comp
-L rdimm-breakout:R_0R_0603 R?
+L rdimm-breakout:R_0R_0603 R12
 U 1 1 623F859E
 P 11225 5850
-F 0 "R?" H 11275 5775 60  0000 C CNN
+F 0 "R12" H 11275 5750 60  0000 C CNN
 F 1 "R_0R_0603" H 11225 5700 60  0001 C CNN
 F 2 "rdimm-breakout-footprints:0603-res" H 11425 6050 60  0001 L CNN
@@
 $EndComp
 $Comp
-L rdimm-breakout:R_10k_0402 R?
+L rdimm-breakout:R_10k_0402 R8
 U 1 1 62412FCB
 P 7275 5250
-F 0 "R?" V 7125 5250 60  0000 L CNN
+F 0 "R8" V 7125 5250 60  0000 L CNN
 F 1 "R_10k_0402" H 7275 5100 60  0001 C CNN
 F 2 "rdimm-breakout-footprints:0402-res" H 7475 5450 60  0001 L CNN
@@
 $EndComp
 $Comp
-L rdimm-breakout:R_10k_0402 R?
+L rdimm-breakout:R_10k_0402 R9
 U 1 1 62414E08
 P 7475 5250
-F 0 "R?" V 7325 5250 60  0000 L CNN
+F 0 "R9" V 7325 5250 60  0000 L CNN
 F 1 "R_10k_0402" H 7475 5100 60  0001 C CNN
 F 2 "rdimm-breakout-footprints:0402-res" H 7675 5450 60  0001 L CNN
@@
 $EndComp
 $Comp
-L rdimm-breakout:R_10k_0402 R?
+L rdimm-breakout:R_10k_0402 R10
 U 1 1 62415065
 P 8625 5275
-F 0 "R?" V 8475 5275 60  0000 L CNN
+F 0 "R10" V 8475 5275 60  0000 L CNN
 F 1 "R_10k_0402" H 8625 5125 60  0001 C CNN
 F 2 "rdimm-breakout-footprints:0402-res" H 8825 5475 60  0001 L CNN
@@
 $EndComp
 $Comp
-L rdimm-breakout:R_10k_0402 R?
+L rdimm-breakout:R_10k_0402 R11
 U 1 1 62415366
 P 8825 5275
-F 0 "R?" V 8675 5275 60  0000 L CNN
+F 0 "R11" V 8675 5275 60  0000 L CNN
 F 1 "R_10k_0402" H 8825 5125 60  0001 C CNN
 F 2 "rdimm-breakout-footprints:0402-res" H 9025 5475 60  0001 L CNN
@@
 	0    1    1    0
 $EndComp
+Text GLabel 7150 5475 0    50   Input ~ 0
+VCC3V3
+Text GLabel 9025 5475 2    50   Input ~ 0
+VCC2V5
+$Comp
+L rdimm-breakout:C_100n_0402 C?
+U 1 1 6249B5B0
+P 6500 5375
+AR Path="/60225B0C/6249B5B0" Ref="C?"  Part="1"
+AR Path="/61B4860C/6249B5B0" Ref="C22"  Part="1"
+F 0 "C22" H 6525 5475 60  0000 L CNN
+F 1 "C_100n_0402" H 6500 5225 60  0001 C CNN
+F 2 "rdimm-breakout-footprints:0402-cap" H 6700 5575 60  0001 L CNN
+F 3 "" H 6500 5375 50  0001 C CNN
+F 4 "Walsin" H 6700 5775 60  0001 L CNN "Manufacturer"
+F 5 "0402X104K6R3CT" H 6700 5675 60  0001 L CNN "MPN"
+F 6 "100n" H 6525 5275 50  0000 L CNN "Val"
+	1    6500 5375
+	1    0    0    -1
+$EndComp
+$Comp
+L rdimm-breakout:GND-rdimm-breakout #PWR?
+U 1 1 6249B5B6
+P 6500 5525
+AR Path="/60225B0C/6249B5B6" Ref="#PWR?"  Part="1"
+AR Path="/61B4860C/6249B5B6" Ref="#PWR0135"  Part="1"
+F 0 "#PWR0135" H 6500 5275 50  0001 C CNN
+F 1 "GND" H 6505 5352 50  0000 C CNN
+F 2 "" H 6500 5525 50  0001 C CNN
+F 3 "" H 6500 5525 50  0001 C CNN
+	1    6500 5525
+	1    0    0    -1
+$EndComp
+$Comp
+L rdimm-breakout:C_100n_0402 C?
+U 1 1 6249F036
+P 9725 5450
+AR Path="/60225B0C/6249F036" Ref="C?"  Part="1"
+AR Path="/61B4860C/6249F036" Ref="C23"  Part="1"
+F 0 "C23" H 9750 5550 60  0000 L CNN
+F 1 "C_100n_0402" H 9725 5300 60  0001 C CNN
+F 2 "rdimm-breakout-footprints:0402-cap" H 9925 5650 60  0001 L CNN
+F 3 "" H 9725 5450 50  0001 C CNN
+F 4 "Walsin" H 9925 5850 60  0001 L CNN "Manufacturer"
+F 5 "0402X104K6R3CT" H 9925 5750 60  0001 L CNN "MPN"
+F 6 "100n" H 9750 5350 50  0000 L CNN "Val"
+	1    9725 5450
+	1    0    0    -1
+$EndComp
+$Comp
+L rdimm-breakout:GND-rdimm-breakout #PWR?
+U 1 1 6249F03C
+P 9725 5600
+AR Path="/60225B0C/6249F03C" Ref="#PWR?"  Part="1"
+AR Path="/61B4860C/6249F03C" Ref="#PWR0136"  Part="1"
+F 0 "#PWR0136" H 9725 5350 50  0001 C CNN
+F 1 "GND" H 9730 5427 50  0000 C CNN
+F 2 "" H 9725 5600 50  0001 C CNN
+F 3 "" H 9725 5600 50  0001 C CNN
+	1    9725 5600
+	1    0    0    -1
+$EndComp
+Text GLabel 6500 5225 1    50   Input ~ 0
+VCC3V3
+Text GLabel 9725 5300 1    50   Input ~ 0
+VCC2V5
+$Comp
+L rdimm-breakout:0022232041 J4
+U 1 1 624BF565
+P 11675 5000
+F 0 "J4" V 11774 4872 50  0000 R CNN
+F 1 "0022232041" V 11865 4872 50  0000 R CNN
+F 2 "rdimm-breakout-footprints:PinHeader_1x4_P2.54mm_Drill1.02mm" H 11875 5200 60  0001 L CNN
+F 3 "https://www.molex.com/pdm_docs/sd/022232041_sd.pdf" H 11875 5300 60  0001 L CNN
+F 4 "0022232041" H 11875 5500 60  0001 L CNN "MPN"
+F 5 "Molex" H 11875 6100 60  0001 L CNN "Manufacturer"
+	1    11675 5000
+	0    -1   1    0
+$EndComp
 $EndSCHEMATC

Commit message: Add initial component placement
Parts:
- J4: footprint rdimm-breakout-footprints:PinHeader_1x4_P2.54mm_Drill1.02mm -> antmicro-footprints:PinHeader_1x4_P2.54mm_Drill1.02mm; symbol rdimm-breakout:0022232041 -> antmicroRectangularConnectorsHeadersMalePins:0022232041
Changed lines of the file:
@@
 VCC2V5
 $Comp
-L rdimm-breakout:0022232041 J4
+L antmicroRectangularConnectorsHeadersMalePins:0022232041 J4
 U 1 1 624BF565
 P 11675 5000
 F 0 "J4" V 11774 4872 50  0000 R CNN
 F 1 "0022232041" V 11865 4872 50  0000 R CNN
-F 2 "rdimm-breakout-footprints:PinHeader_1x4_P2.54mm_Drill1.02mm" H 11875 5200 60  0001 L CNN
+F 2 "antmicro-footprints:PinHeader_1x4_P2.54mm_Drill1.02mm" H 11875 5200 60  0001 L CNN
 F 3 "https://www.molex.com/pdm_docs/sd/022232041_sd.pdf" H 11875 5300 60  0001 L CNN
 F 4 "0022232041" H 11875 5500 60  0001 L CNN "MPN"

Commit message: Bump rev to 1.0.1
Parts:
- J4: footprint antmicro-footprints:PinHeader_1x4_P2.54mm_Drill1.02mm -> rdimm-breakout-footprints:PinHeader_1x4_P2.54mm_Drill1.02mm; symbol antmicroRectangularConnectorsHeadersMalePins:0022232041 -> rdimm-breakout:0022232041
Changed lines of the file:
@@
 Sheet 4 4
 Title "RDIMM-breakout"
-Date "2021-09"
-Rev "1.0.0"
+Date "2021-10"
+Rev "1.0.1"
 Comp "Antmicro Ltd."
 Comment1 "www.antmicro.com"
@@
 VCC2V5
 $Comp
-L antmicroRectangularConnectorsHeadersMalePins:0022232041 J4
+L rdimm-breakout:0022232041 J4
 U 1 1 624BF565
 P 11675 5000
 F 0 "J4" V 11774 4872 50  0000 R CNN
 F 1 "0022232041" V 11865 4872 50  0000 R CNN
-F 2 "antmicro-footprints:PinHeader_1x4_P2.54mm_Drill1.02mm" H 11875 5200 60  0001 L CNN
+F 2 "rdimm-breakout-footprints:PinHeader_1x4_P2.54mm_Drill1.02mm" H 11875 5200 60  0001 L CNN
 F 3 "https://www.molex.com/pdm_docs/sd/022232041_sd.pdf" H 11875 5300 60  0001 L CNN
 F 4 "0022232041" H 11875 5500 60  0001 L CNN "MPN"
