File: fpga-banks-16-34.sch (KiCad schematic (older format))
At the start: 19 parts, among them J4 0022232041, U8 PCA9517ADMR2G

Commit message: Update naming convention
Parts:
- C22, C23: footprint rdimm-breakout-footprints:0402-cap -> ddr4-spd-breakout-footprints:0402-cap; symbol rdimm-breakout:C_100n_0402 -> ddr4-spd-breakout:C_100n_0402
- J4: footprint rdimm-breakout-footprints:PinHeader_1x4_P2.54mm_Drill1.02mm -> ddr4-spd-breakout-footprints:PinHeader_1x4_P2.54mm_Drill1.02mm; symbol rdimm-breakout:0022232041 -> ddr4-spd-breakout:0022232041
- R10, R11, R8, R9: footprint rdimm-breakout-footprints:0402-res -> ddr4-spd-breakout-footprints:0402-res; symbol rdimm-breakout:R_10k_0402 -> ddr4-spd-breakout:R_10k_0402
- R12: footprint rdimm-breakout-footprints:0603-res -> ddr4-spd-breakout-footprints:0603-res; symbol rdimm-breakout:R_0R_0603 -> ddr4-spd-breakout:R_0R_0603
- R164, R165, R166, R167, R168, R169: footprint rdimm-breakout-footprints:0402-res -> ddr4-spd-breakout-footprints:0402-res; symbol rdimm-breakout:R_0R_0402-rdimm-breakout -> ddr4-spd-breakout:R_0R_0402-ddr4-spd-breakout
- R170: footprint rdimm-breakout-footprints:0402-res -> ddr4-spd-breakout-footprints:0402-res; symbol rdimm-breakout:R_4k7_0402-rdimm-breakout -> ddr4-spd-breakout:R_4k7_0402-ddr4-spd-breakout
- TP1, TP12, TP2: footprint rdimm-breakout-footprints:Testpoint_smd_1mm -> ddr4-spd-breakout-footprints:Testpoint_smd_1mm; symbol rdimm-breakout:TP_SMD1MM-rdimm-breakout -> ddr4-spd-breakout:TP_SMD1MM-ddr4-spd-breakout
- U8: footprint rdimm-breakout-footprints:TSSOP-8_W3mm -> ddr4-spd-breakout-footprints:TSSOP-8_W3mm; symbol rdimm-breakout:PCA9517ADMR2G-rdimm-breakout -> ddr4-spd-breakout:PCA9517ADMR2G-ddr4-spd-breakout
Changed lines of the file:
@@
 ~EVENT
 $Comp
-L rdimm-breakout:R_4k7_0402-rdimm-breakout R170
+L ddr4-spd-breakout:R_4k7_0402-ddr4-spd-breakout R170
 U 1 1 628AFA47
 P 3650 5750
 F 0 "R170" V 3500 5775 60  0000 L CNN
 F 1 "R_4k7_0402" H 3650 5600 60  0001 C CNN
-F 2 "rdimm-breakout-footprints:0402-res" H 3850 5950 60  0001 L CNN
+F 2 "ddr4-spd-breakout-footprints:0402-res" H 3850 5950 60  0001 L CNN
 F 3 "" H 3650 5750 50  0001 C CNN
 F 4 "VISHAY" H 3850 6150 60  0001 L CNN "Manufacturer"
@@
 	5375 6025 5375 6075
 $Comp
-L rdimm-breakout:R_0R_0402-rdimm-breakout R168
+L ddr4-spd-breakout:R_0R_0402-ddr4-spd-breakout R168
 U 1 1 622013A9
 P 5725 5550
 F 0 "R168" H 5425 5650 60  0000 L CNN
 F 1 "R_0R_0402" H 5725 5400 60  0001 C CNN
-F 2 "rdimm-breakout-footprints:0402-res" H 5925 5750 60  0001 L CNN
+F 2 "ddr4-spd-breakout-footprints:0402-res" H 5925 5750 60  0001 L CNN
 F 3 "" H 5725 5550 50  0001 C CNN
 F 4 "PANASONIC" H 5925 5950 60  0001 L CNN "Manufacturer"
@@
 $EndComp
 $Comp
-L rdimm-breakout:R_0R_0402-rdimm-breakout R166
+L ddr4-spd-breakout:R_0R_0402-ddr4-spd-breakout R166
 U 1 1 62200AC4
 P 5550 5550
 F 0 "R166" H 5250 5650 60  0000 L CNN
 F 1 "R_0R_0402" H 5550 5400 60  0001 C CNN
-F 2 "rdimm-breakout-footprints:0402-res" H 5750 5750 60  0001 L CNN
+F 2 "ddr4-spd-breakout-footprints:0402-res" H 5750 5750 60  0001 L CNN
 F 3 "" H 5550 5550 50  0001 C CNN
 F 4 "PANASONIC" H 5750 5950 60  0001 L CNN "Manufacturer"
@@
 $EndComp
 $Comp
-L rdimm-breakout:R_0R_0402-rdimm-breakout R164
+L ddr4-spd-breakout:R_0R_0402-ddr4-spd-breakout R164
 U 1 1 621FEF1F
 P 5375 5550
 F 0 "R164" H 5075 5650 60  0000 L CNN
 F 1 "R_0R_0402" H 5375 5400 60  0001 C CNN
-F 2 "rdimm-breakout-footprints:0402-res" H 5575 5750 60  0001 L CNN
+F 2 "ddr4-spd-breakout-footprints:0402-res" H 5575 5750 60  0001 L CNN
 F 3 "" H 5375 5550 50  0001 C CNN
 F 4 "PANASONIC" H 5575 5950 60  0001 L CNN "Manufacturer"
@@
 $EndComp
 $Comp
-L rdimm-breakout:GND-rdimm-breakout #PWR0266
+L ddr4-spd-breakout:GND-ddr4-spd-breakout #PWR0266
 U 1 1 621A4B23
 P 5725 6375
@@
 $EndComp
 $Comp
-L rdimm-breakout:GND-rdimm-breakout #PWR0265
+L ddr4-spd-breakout:GND-ddr4-spd-breakout #PWR0265
 U 1 1 621A3D5D
 P 5550 6375
@@
 $EndComp
 $Comp
-L rdimm-breakout:GND-rdimm-breakout #PWR0146
+L ddr4-spd-breakout:GND-ddr4-spd-breakout #PWR0146
 U 1 1 621A348D
 P 5375 6375
@@
 $EndComp
 $Comp
-L rdimm-breakout:R_0R_0402-rdimm-breakout R169
+L ddr4-spd-breakout:R_0R_0402-ddr4-spd-breakout R169
 U 1 1 6200BC51
 P 5725 6225
 F 0 "R169" H 5425 6325 60  0000 L CNN
 F 1 "R_0R_0402" H 5725 6075 60  0001 C CNN
-F 2 "rdimm-breakout-footprints:0402-res" H 5925 6425 60  0001 L CNN
+F 2 "ddr4-spd-breakout-footprints:0402-res" H 5925 6425 60  0001 L CNN
 F 3 "" H 5725 6225 50  0001 C CNN
 F 4 "PANASONIC" H 5925 6625 60  0001 L CNN "Manufacturer"
@@
 $EndComp
 $Comp
-L rdimm-breakout:R_0R_0402-rdimm-breakout R167
+L ddr4-spd-breakout:R_0R_0402-ddr4-spd-breakout R167
 U 1 1 6200B3D4
 P 5550 6225
 F 0 "R167" H 5250 6325 60  0000 L CNN
 F 1 "R_0R_0402" H 5550 6075 60  0001 C CNN
-F 2 "rdimm-breakout-footprints:0402-res" H 5750 6425 60  0001 L CNN
+F 2 "ddr4-spd-breakout-footprints:0402-res" H 5750 6425 60  0001 L CNN
 F 3 "" H 5550 6225 50  0001 C CNN
 F 4 "PANASONIC" H 5750 6625 60  0001 L CNN "Manufacturer"
@@
 $EndComp
 $Comp
-L rdimm-breakout:R_0R_0402-rdimm-breakout R165
+L ddr4-spd-breakout:R_0R_0402-ddr4-spd-breakout R165
 U 1 1 61FD65FE
 P 5375 6225
 F 0 "R165" H 5075 6325 60  0000 L CNN
 F 1 "R_0R_0402" H 5375 6075 60  0001 C CNN
-F 2 "rdimm-breakout-footprints:0402-res" H 5575 6425 60  0001 L CNN
+F 2 "ddr4-spd-breakout-footprints:0402-res" H 5575 6425 60  0001 L CNN
 F 3 "" H 5375 6225 50  0001 C CNN
 F 4 "PANASONIC" H 5575 6625 60  0001 L CNN "Manufacturer"
@@
 	8425 5775 8600 5775
 $Comp
-L rdimm-breakout:TP_SMD1MM-rdimm-breakout TP12
+L ddr4-spd-breakout:TP_SMD1MM-ddr4-spd-breakout TP12
 U 1 1 61DDE955
 P 8700 5775
 F 0 "TP12" V 8700 5725 50  0000 R CNN
 F 1 "TP_SMD1MM" H 8700 5675 50  0001 C CNN
-F 2 "rdimm-breakout-footprints:Testpoint_smd_1mm" H 8900 5975 60  0001 L CNN
+F 2 "ddr4-spd-breakout-footprints:Testpoint_smd_1mm" H 8900 5975 60  0001 L CNN
 F 3 "" H 8900 6075 60  0001 L CNN
 	1    8700 5775
@@
 	8425 5675 8625 5675
 $Comp
-L rdimm-breakout:PCA9517ADMR2G-rdimm-breakout U8
+L ddr4-spd-breakout:PCA9517ADMR2G-ddr4-spd-breakout U8
 U 1 1 61682D3C
 P 8125 5775
 F 0 "U8" H 8075 6362 60  0000 C CNN
 F 1 "PCA9517ADMR2G" H 8075 6256 60  0000 C CNN
-F 2 "rdimm-breakout-footprints:TSSOP-8_W3mm" H 8425 6225 60  0001 L CNN
+F 2 "ddr4-spd-breakout-footprints:TSSOP-8_W3mm" H 8425 6225 60  0001 L CNN
 F 3 "" H 8375 6325 60  0001 L CNN
 F 4 "PCA9517ADMR2G" H 8375 6425 60  0001 L CNN "MPN"
@@
 $EndComp
 $Comp
-L rdimm-breakout:GND-rdimm-breakout #PWR0145
+L ddr4-spd-breakout:GND-ddr4-spd-breakout #PWR0145
 U 1 1 6227AF37
 P 7550 5775
@@
 I2C header
 $Comp
-L rdimm-breakout:TP_SMD1MM-rdimm-breakout TP2
+L ddr4-spd-breakout:TP_SMD1MM-ddr4-spd-breakout TP2
 U 1 1 61B53CB4
 P 10875 5300
 F 0 "TP2" V 10875 5250 50  0000 R CNN
 F 1 "TP_SMD1MM" H 10875 5200 50  0001 C CNN
-F 2 "rdimm-breakout-footprints:Testpoint_smd_1mm" H 11075 5500 60  0001 L CNN
+F 2 "ddr4-spd-breakout-footprints:Testpoint_smd_1mm" H 11075 5500 60  0001 L CNN
 F 3 "" H 11075 5600 60  0001 L CNN
 	1    10875 5300
@@
 	10875 5200 10800 5200
 $Comp
-L rdimm-breakout:TP_SMD1MM-rdimm-breakout TP1
+L ddr4-spd-breakout:TP_SMD1MM-ddr4-spd-breakout TP1
 U 1 1 61B5478E
 P 10875 5000
 F 0 "TP1" V 10875 4950 50  0000 R CNN
 F 1 "TP_SMD1MM" H 10875 4900 50  0001 C CNN
-F 2 "rdimm-breakout-footprints:Testpoint_smd_1mm" H 11075 5200 60  0001 L CNN
+F 2 "ddr4-spd-breakout-footprints:Testpoint_smd_1mm" H 11075 5200 60  0001 L CNN
 F 3 "" H 11075 5300 60  0001 L CNN
 	1    10875 5000
@@
 	11400 5300 11575 5300
 $Comp
-L rdimm-breakout:GND-rdimm-breakout #PWR0134
+L ddr4-spd-breakout:GND-ddr4-spd-breakout #PWR0134
 U 1 1 623664C2
 P 11400 5300
@@
 V_AUX
 $Comp
-L rdimm-breakout:R_0R_0603 R12
+L ddr4-spd-breakout:R_0R_0603 R12
 U 1 1 623F859E
 P 11225 5850
 F 0 "R12" H 11275 5750 60  0000 C CNN
 F 1 "R_0R_0603" H 11225 5700 60  0001 C CNN
-F 2 "rdimm-breakout-footprints:0603-res" H 11425 6050 60  0001 L CNN
+F 2 "ddr4-spd-breakout-footprints:0603-res" H 11425 6050 60  0001 L CNN
 F 3 "" H 11225 5850 50  0001 C CNN
 F 4 "BOURNS" H 11425 6250 60  0001 L CNN "Manufacturer"
@@
 $EndComp
 $Comp
-L rdimm-breakout:R_10k_0402 R8
+L ddr4-spd-breakout:R_10k_0402 R8
 U 1 1 62412FCB
 P 7275 5250
 F 0 "R8" V 7125 5250 60  0000 L CNN
 F 1 "R_10k_0402" H 7275 5100 60  0001 C CNN
-F 2 "rdimm-breakout-footprints:0402-res" H 7475 5450 60  0001 L CNN
+F 2 "ddr4-spd-breakout-footprints:0402-res" H 7475 5450 60  0001 L CNN
 F 3 "" H 7275 5250 50  0001 C CNN
 F 4 "VISHAY" H 7475 5650 60  0001 L CNN "Manufacturer"
@@
 $EndComp
 $Comp
-L rdimm-breakout:R_10k_0402 R9
+L ddr4-spd-breakout:R_10k_0402 R9
 U 1 1 62414E08
 P 7475 5250
 F 0 "R9" V 7325 5250 60  0000 L CNN
 F 1 "R_10k_0402" H 7475 5100 60  0001 C CNN
-F 2 "rdimm-breakout-footprints:0402-res" H 7675 5450 60  0001 L CNN
+F 2 "ddr4-spd-breakout-footprints:0402-res" H 7675 5450 60  0001 L CNN
 F 3 "" H 7475 5250 50  0001 C CNN
 F 4 "VISHAY" H 7675 5650 60  0001 L CNN "Manufacturer"
@@
 $EndComp
 $Comp
-L rdimm-breakout:R_10k_0402 R10
+L ddr4-spd-breakout:R_10k_0402 R10
 U 1 1 62415065
 P 8625 5275
 F 0 "R10" V 8475 5275 60  0000 L CNN
 F 1 "R_10k_0402" H 8625 5125 60  0001 C CNN
-F 2 "rdimm-breakout-footprints:0402-res" H 8825 5475 60  0001 L CNN
+F 2 "ddr4-spd-breakout-footprints:0402-res" H 8825 5475 60  0001 L CNN
 F 3 "" H 8625 5275 50  0001 C CNN
 F 4 "VISHAY" H 8825 5675 60  0001 L CNN "Manufacturer"
@@
 $EndComp
 $Comp
-L rdimm-breakout:R_10k_0402 R11
+L ddr4-spd-breakout:R_10k_0402 R11
 U 1 1 62415366
 P 8825 5275
 F 0 "R11" V 8675 5275 60  0000 L CNN
 F 1 "R_10k_0402" H 8825 5125 60  0001 C CNN
-F 2 "rdimm-breakout-footprints:0402-res" H 9025 5475 60  0001 L CNN
+F 2 "ddr4-spd-breakout-footprints:0402-res" H 9025 5475 60  0001 L CNN
 F 3 "" H 8825 5275 50  0001 C CNN
 F 4 "VISHAY" H 9025 5675 60  0001 L CNN "Manufacturer"
@@
 VCC2V5
 $Comp
-L rdimm-breakout:C_100n_0402 C?
+L ddr4-spd-breakout:C_100n_0402 C?
 U 1 1 6249B5B0
 P 6500 5375
@@
 F 0 "C22" H 6525 5475 60  0000 L CNN
 F 1 "C_100n_0402" H 6500 5225 60  0001 C CNN
-F 2 "rdimm-breakout-footprints:0402-cap" H 6700 5575 60  0001 L CNN
+F 2 "ddr4-spd-breakout-footprints:0402-cap" H 6700 5575 60  0001 L CNN
 F 3 "" H 6500 5375 50  0001 C CNN
 F 4 "Walsin" H 6700 5775 60  0001 L CNN "Manufacturer"
@@
 $EndComp
 $Comp
-L rdimm-breakout:GND-rdimm-breakout #PWR?
+L ddr4-spd-breakout:GND-ddr4-spd-breakout #PWR?
 U 1 1 6249B5B6
 P 6500 5525
@@
 $EndComp
 $Comp
-L rdimm-breakout:C_100n_0402 C?
+L ddr4-spd-breakout:C_100n_0402 C?
 U 1 1 6249F036
 P 9725 5450
@@
 F 0 "C23" H 9750 5550 60  0000 L CNN
 F 1 "C_100n_0402" H 9725 5300 60  0001 C CNN
-F 2 "rdimm-breakout-footprints:0402-cap" H 9925 5650 60  0001 L CNN
+F 2 "ddr4-spd-breakout-footprints:0402-cap" H 9925 5650 60  0001 L CNN
 F 3 "" H 9725 5450 50  0001 C CNN
 F 4 "Walsin" H 9925 5850 60  0001 L CNN "Manufacturer"
@@
 $EndComp
 $Comp
-L rdimm-breakout:GND-rdimm-breakout #PWR?
+L ddr4-spd-breakout:GND-ddr4-spd-breakout #PWR?
 U 1 1 6249F03C
 P 9725 5600
@@
 VCC2V5
 $Comp
-L rdimm-breakout:0022232041 J4
+L ddr4-spd-breakout:0022232041 J4
 U 1 1 624BF565
 P 11675 5000
 F 0 "J4" V 11774 4872 50  0000 R CNN
 F 1 "0022232041" V 11865 4872 50  0000 R CNN
-F 2 "rdimm-breakout-footprints:PinHeader_1x4_P2.54mm_Drill1.02mm" H 11875 5200 60  0001 L CNN
+F 2 "ddr4-spd-breakout-footprints:PinHeader_1x4_P2.54mm_Drill1.02mm" H 11875 5200 60  0001 L CNN
 F 3 "https://www.molex.com/pdm_docs/sd/022232041_sd.pdf" H 11875 5300 60  0001 L CNN
 F 4 "0022232041" H 11875 5500 60  0001 L CNN "MPN"
